File: pcb/RCC.kicad_sch (KiCad schematic)
At the start: 15 parts, among them SW1 SW_MEC_5E, U1 ATtiny402-SS

Commit message: Change value of R3
Parts:
- R3: value 1Meg -> 10k; VendorId 102999 -> 102967
Changed lines of the file:
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@@
       (effects (font (size 1.27 1.27)) (justify left))
     )
-    (property "Value" "1Meg" (at 175.26 96.52 0)
+    (property "Value" "10k" (at 175.26 96.52 0)
       (effects (font (size 1.27 1.27)) (justify left))
     )
@@
       (effects (font (size 1.27 1.27)) hide)
     )
-    (property "VendorId" "102999" (at 172.72 95.25 0)
+    (property "VendorId" "102967" (at 172.72 95.25 0)
       (effects (font (size 1.27 1.27)) hide)
     )
