File: pcb/RCC.kicad_sch (KiCad schematic)
At the start: 15 parts, among them SW1 SW_MEC_5E, U1 ATtiny402-SS

Commit message: Change partlist vendors
Parts:
- D1, D2: Vendor DigiKey -> HTL; VendorId 3147-T3A33BRG-H9C0002X1U1930CT-ND -> 103607
- U1: VendorId ATTINY402-SSNRCT-ND -> 103608
Changed lines of the file:
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@@
       (effects (font (size 1.27 1.27)) (justify left top) hide)
     )
-    (property "Vendor" "DigiKey" (at 220.98 81.28 0)
-      (effects (font (size 1.27 1.27)) hide)
-    )
-    (property "VendorId" "3147-T3A33BRG-H9C0002X1U1930CT-ND" (at 220.98 81.28 0)
+    (property "Vendor" "HTL" (at 220.98 81.28 0)
+      (effects (font (size 1.27 1.27)) hide)
+    )
+    (property "VendorId" "103607" (at 220.98 81.28 0)
       (effects (font (size 1.27 1.27)) hide)
     )
@@
       (effects (font (size 1.27 1.27)) (justify left top) hide)
     )
-    (property "Vendor" "DigiKey" (at 203.2 81.28 0)
-      (effects (font (size 1.27 1.27)) hide)
-    )
-    (property "VendorId" "3147-T3A33BRG-H9C0002X1U1930CT-ND" (at 203.2 81.28 0)
+    (property "Vendor" "HTL" (at 203.2 81.28 0)
+      (effects (font (size 1.27 1.27)) hide)
+    )
+    (property "VendorId" "103607" (at 203.2 81.28 0)
       (effects (font (size 1.27 1.27)) hide)
     )
@@
       (effects (font (size 1.27 1.27)) hide)
     )
-    (property "VendorId" "ATTINY402-SSNRCT-ND" (at 146.05 83.82 0)
-      (effects (font (size 1.27 1.27)) hide)
-    )
+    (property "VendorId" "103608" (at 146.05 83.82 0)
+      (effects (font (size 1.27 1.27)) hide)
+    )
